File: docs/door monitor.kicad_pcb (KiCad board)
At the start: 2 copper layers, 48.9 x 30.5 mm, 11 parts, among them J1 USB_B_Mini, J2 Screw_Terminal_01x02, SW1 SW_Push, U1 LM2937xS, U2 ESP-01v090

Commit message: Update electrical shema
Parts:
- added D1: LED, LED_SMD:LED_0805_2012Metric_Pad1.15x1.40mm_HandSolder, F.Cu at (154.2, 73.7)
- added J3: Conn_01x02_Male, Connector_PinHeader_2.54mm:PinHeader_1x02_P2.54mm_Horizontal, B.Cu at (144.8, 73.7)
- added J4: Conn_01x02_Male, Connector_PinHeader_2.54mm:PinHeader_1x02_P2.54mm_Horizontal, B.Cu at (158.8, 76.2)
- added R5: R, Resistor_SMD:R_0805_2012Metric_Pad1.15x1.40mm_HandSolder, F.Cu at (149.4, 73.7)
- C2: footprint Capacitor_THT:CP_Radial_D4.0mm_P2.00mm -> Capacitor_THT:CP_Radial_D5.0mm_P2.50mm
Routing:
- net Net-(D1-Pad2): track 0.00 -> 7.59 mm
- net Net-(D1-Pad1): track 0.00 -> 2.78 mm
- net Earth: track 0.25 -> 2.91 mm
- added copper zone on F.Cu, net Net-(D1-Pad2)
- added copper zone on F.Cu, net Net-(J3-Pad2)
Other:
- board size 48.9 x 30.5 mm -> 48.9 x 43.8 mm
